Commit message: Update TEST_PROJECT_VIMAL.xacro

File: urdf_vimal/TEST_PROJECT_VIMAL_description/urdf/TEST_PROJECT_VIMAL.xacro (robot description, xacro)
@@ -108,5 +108,5 @@
   <parent link="base_link"/>
   <child link="right_whell_1"/>
-  <axis xyz="-0.0 1.0 -0.0"/>
+  <axis xyz="0.0 1.0 0.0"/>
 </joint>
 <joint name="Rev2" type="continuous">
@@ -114,5 +114,5 @@
   <parent link="base_link"/>
   <child link="left_whell_1"/>
-  <axis xyz="-0.0 1.0 -0.0"/>
+  <axis xyz="0.0 1.0 0.0"/>
 </joint>
 <joint name="Rev3" type="continuous">
@@ -120,5 +120,5 @@
   <parent link="_mount_1"/>
   <child link="lidar_1"/>
-  <axis xyz="0.0 -0.0 1.0"/>
+  <axis xyz="0.0 0.0 1.0"/>
 </joint>
 <joint name="Rigid4" type="fixed">
